File: kicad/rnode_dip/rnode_dip.sch (KiCad schematic (older format))
At the start: 1 part

Commit message: update
Parts:
- added C? (x6): C, symbol Device:C
- added J?: Conn_01x06_Male, symbol Connector:Conn_01x06_Male
- added J?: AVR-ISP-6, symbol Connector:AVR-ISP-6
- added R?: R, symbol Device:R
- added SW?: SW_Push_Dual, symbol Switch:SW_Push_Dual
- added U?: MCP1700-3302E_TO92, Package_TO_SOT_THT:TO-92_Inline, symbol Regulator_Linear:MCP1700-3302E_TO92
- added U?: RFM95HW, mysensors_radios:RFM69HW_SMD_ThroughHole_Handsoldering, symbol mysensors_radios:RFM95HW
- added Y?: Crystal, symbol Device:Crystal
Connections:
- net VCC: now reaches U?.10 (VCC)
- net VCC: now also U?.30 (AVCC), C?.1, C?.1, R?.2, U?.3 (VO)
- net GND: now reaches U?.11 (GND), U?.31 (GND)
- net GND: now also C?.2, C?.2, C?.2, C?.2, C?.2, J?.1 (Pin_1), SW?.3, SW?.4, U?.1 (GND)
- net at U?.12 (XTAL2): now also C?.1, Y?.2
- net at U?.13 (XTAL1): now also C?.1, Y?.1
- net UART_RX0: now reaches U?.14 (PD0)
- net UART_RX0: now also J?.4 (Pin_4)
- net UART_TX0: now reaches U?.15 (PD1)
- net UART_TX0: now also J?.5 (Pin_5)
- net UART_RX1: now reaches U?.16 (PD2)
- net UART_TX1: now reaches U?.17 (PD3)
- net RESET: now reaches U?.9 (~RESET)
- net RESET: now also C?.1, R?.1, SW?.1, SW?.2
- new net: C?.2, J?.6 (Pin_6)
- new net VBUS: C?.1, J?.3 (Pin_3), U?.2 (VI)
Other:
- note added: "FTDI"
- note added: "ISP"
- note added: "LDO"
- note added: "RESET"
- moved on the sheet: U?

Commit message: update
Parts:
- added J?: INAIR_L, symbol Connector:Conn_01x07_Female
- added J?: INAIR_R, symbol Connector:Conn_01x07_Female
Connections:
- net VCC is gone; now on net +3V3: C?.1, C?.1, R?.2, U?.10 (VCC), U?.3 (VO), U?.30 (AVCC)
- net GND: now also J?.6 (GND), J?.7 (Pin_7)
- net RESET: now also J?.5 (~RST)
- net VBUS: now also J?.2 (VCC)
- net DIO_0: now reaches U?.3 (PB2)
- net DIO_0: now also U?.14 (DIO0), J?.3 (Pin_3)
- net LORA_RST: now reaches U?.4 (PB3)
- net LORA_RST: now also U?.6 (RESET), J?.4 (Pin_4)
- net LORA_CS: now reaches U?.5 (PB4)
- net LORA_CS: now also U?.5 (NSS), J?.6 (Pin_6)
- net MOSI: now reaches U?.6 (PB5)
- net MOSI: now also J?.4 (MOSI), U?.3 (MOSI), J?.3 (Pin_3)
- net MISO: now reaches U?.7 (PB6)
- net MISO: now also J?.1 (MISO), U?.2 (MISO), J?.4 (Pin_4)
- net SCK: now reaches U?.8 (PB7)
- net SCK: now also J?.3 (SCK), U?.4 (SCK), J?.5 (Pin_5)
- net +3V3: now reaches U?.13 (3.3V)
- net +3V3: now also J?.6 (Pin_6)
Other:
- note added: "LORA"
- moved on the sheet: U?
Changed lines of the file:
@@
 	1600 6850 1100 6850
 Connection ~ 1600 6850
-$Comp
-L power:VCC #PWR?
-U 1 1 602FFF7F
-P 3800 6850
-F 0 "#PWR?" H 3800 6700 50  0001 C CNN
-F 1 "VCC" H 3817 7023 50  0000 C CNN
-F 2 "" H 3800 6850 50  0001 C CNN
-F 3 "" H 3800 6850 50  0001 C CNN
-	1    3800 6850
-	1    0    0    -1
-$EndComp
 Wire Wire Line
 	3800 6850 3250 6850
@@
 	4050 1750 4050 1550
 $Comp
-L power:VCC #PWR?
-U 1 1 6034FFC2
-P 2450 1250
-F 0 "#PWR?" H 2450 1100 50  0001 C CNN
-F 1 "VCC" H 2467 1423 50  0000 C CNN
-F 2 "" H 2450 1250 50  0001 C CNN
-F 3 "" H 2450 1250 50  0001 C CNN
-	1    2450 1250
-	1    0    0    -1
-$EndComp
-$Comp
 L Device:C C?
 U 1 1 603504A9
@@
 L mysensors_radios:RFM95HW U?
 U 1 1 603D7158
-P 10150 2950
-F 0 "U?" H 10150 3564 40  0000 C CNN
-F 1 "RFM95HW" H 10150 3488 40  0000 C CNN
-F 2 "mysensors_radios:RFM69HW_SMD_ThroughHole_Handsoldering" H 10150 2950 30  0001 C CIN
-F 3 "rfm95" H 10150 3397 60  0000 C CNN
-	1    10150 2950
+P 10100 4500
+F 0 "U?" H 9800 4950 40  0000 C CNN
+F 1 "RFM95HW" H 9800 4850 40  0000 C CNN
+F 2 "mysensors_radios:RFM69HW_SMD_ThroughHole_Handsoldering" H 10100 4500 30  0001 C CIN
+F 3 "rfm95" H 10100 4400 60  0000 C CNN
+	1    10100 4500
 	1    0    0    -1
 $EndComp
@@
 	1    0    0    -1
 $EndComp
-$Comp
-L power:VCC #PWR?
-U 1 1 603E6D3F
+Wire Wire Line
+	5250 1450 5150 1450
+Wire Wire Line
+	5150 1450 5150 1050
+Connection ~ 5150 1450
+$Comp
+L Connector:Conn_01x07_Female J?
+U 1 1 603F5459
+P 8050 4300
+F 0 "J?" H 7942 3775 50  0000 C CNN
+F 1 "INAIR_L" H 7942 3866 50  0000 C CNN
+F 2 "" H 8050 4300 50  0001 C CNN
+F 3 "~" H 8050 4300 50  0001 C CNN
+	1    8050 4300
+	-1   0    0    1
+$EndComp
+$Comp
+L Connector:Conn_01x07_Female J?
+U 1 1 603F7BAF
+P 8050 5450
+F 0 "J?" H 7942 4925 50  0000 C CNN
+F 1 "INAIR_R" H 7942 5016 50  0000 C CNN
+F 2 "" H 8050 5450 50  0001 C CNN
+F 3 "~" H 8050 5450 50  0001 C CNN
+	1    8050 5450
+	-1   0    0    1
+$EndComp
+$Comp
+L power:GND #PWR?
+U 1 1 603FBF93
+P 8450 3750
+F 0 "#PWR?" H 8450 3500 50  0001 C CNN
+F 1 "GND" H 8455 3577 50  0000 C CNN
+F 2 "" H 8450 3750 50  0001 C CNN
+F 3 "" H 8450 3750 50  0001 C CNN
+	1    8450 3750
+	-1   0    0    1
+$EndComp
+$Comp
+L power:+3V3 #PWR?
+U 1 1 60405A81
+P 3800 6850
+F 0 "#PWR?" H 3800 6700 50  0001 C CNN
+F 1 "+3V3" H 3815 7023 50  0000 C CNN
+F 2 "" H 3800 6850 50  0001 C CNN
+F 3 "" H 3800 6850 50  0001 C CNN
+	1    3800 6850
+	1    0    0    -1
+$EndComp
+$Comp
+L power:+3V3 #PWR?
+U 1 1 60406B29
+P 2450 1250
+F 0 "#PWR?" H 2450 1100 50  0001 C CNN
+F 1 "+3V3" H 2465 1423 50  0000 C CNN
+F 2 "" H 2450 1250 50  0001 C CNN
+F 3 "" H 2450 1250 50  0001 C CNN
+	1    2450 1250
+	1    0    0    -1
+$EndComp
+$Comp
+L power:+3V3 #PWR?
+U 1 1 6040C6F5
 P 5150 1050
 F 0 "#PWR?" H 5150 900 50  0001 C CNN
-F 1 "VCC" H 5167 1223 50  0000 C CNN
+F 1 "+3V3" H 5165 1223 50  0000 C CNN
 F 2 "" H 5150 1050 50  0001 C CNN
 F 3 "" H 5150 1050 50  0001 C CNN
@@
 	1    0    0    -1
 $EndComp
-Wire Wire Line
-	5250 1450 5150 1450
-Wire Wire Line
-	5150 1450 5150 1050
-Connection ~ 5150 1450
+$Comp
+L power:+3V3 #PWR?
+U 1 1 604176B3
+P 8550 5150
+F 0 "#PWR?" H 8550 5000 50  0001 C CNN
+F 1 "+3V3" H 8565 5323 50  0000 C CNN
+F 2 "" H 8550 5150 50  0001 C CNN
+F 3 "" H 8550 5150 50  0001 C CNN
+	1    8550 5150
+	1    0    0    -1
+$EndComp
+Wire Wire Line
+	8250 4000 8450 4000
+Wire Wire Line
+	8450 4000 8450 3750
+Wire Wire Line
+	8250 5250 8550 5250
+Wire Wire Line
+	8550 5250 8550 5150
+Text GLabel 8250 5350 2    50   Input ~ 0
+SCK
+Text GLabel 8250 5450 2    50   Input ~ 0
+MISO
+Text GLabel 8250 5550 2    50   Input ~ 0
+MOSI
+Text GLabel 8250 4400 2    50   Input ~ 0
+DIO_0
+Text GLabel 8250 4300 2    50   Input ~ 0
+LORA_RST
+Text GLabel 8250 4100 2    50   Input ~ 0
+LORA_CS
+Text GLabel 9550 4550 0    50   Input ~ 0
+LORA_CS
+Text GLabel 9550 5050 0    50   Input ~ 0
+LORA_RST
+Text GLabel 10650 4500 2    50   Input ~ 0
+DIO_0
+Text GLabel 9550 4750 0    50   Input ~ 0
+MISO
+Text GLabel 9550 4650 0    50   Input ~ 0
+MOSI
+Text GLabel 9550 4850 0    50   Input ~ 0
+SCK
+Text GLabel 10000 1650 2    50   Input ~ 0
+MOSI
+Text GLabel 10000 1550 2    50   Input ~ 0
+MISO
+Text GLabel 10000 1750 2    50   Input ~ 0
+SCK
+Text GLabel 10000 1850 2    50   Input ~ 0
+RESET
+$Comp
+L power:GND #PWR?
+U 1 1 6044E968
+P 9500 2150
+F 0 "#PWR?" H 9500 1900 50  0001 C CNN
+F 1 "GND" H 9505 1977 50  0000 C CNN
+F 2 "" H 9500 2150 50  0001 C CNN
+F 3 "" H 9500 2150 50  0001 C CNN
+	1    9500 2150
+	1    0    0    -1
+$EndComp
+Text GLabel 9500 1250 0    50   Input ~ 0
+VBUS
+$Comp
+L power:+3V3 #PWR?
+U 1 1 6045AC5D
+P 10100 4150
+F 0 "#PWR?" H 10100 4000 50  0001 C CNN
+F 1 "+3V3" H 10250 4200 50  0000 C CNN
+F 2 "" H 10100 4150 50  0001 C CNN
+F 3 "" H 10100 4150 50  0001 C CNN
+	1    10100 4150
+	1    0    0    -1
+$EndComp
+Text GLabel 5750 3350 2    50   Input ~ 0
+SCK
+Text GLabel 5750 3250 2    50   Input ~ 0
+MISO
+Text GLabel 5750 3150 2    50   Input ~ 0
+MOSI
+Text GLabel 5750 3050 2    50   Input ~ 0
+LORA_CS
+Text GLabel 5750 2950 2    50   Input ~ 0
+LORA_RST
+Text GLabel 5750 2850 2    50   Input ~ 0
+DIO_0
+Wire Notes Line
+	11250 3200 7700 3200
+Wire Notes Line
+	7700 3200 7700 6500
+Text Notes 9400 3500 0    118  ~ 0
+LORA
 $EndSCHEMATC
